File: P8000_WDC_Emulator/Hardware/P8000_WDC_Emulator.kicad_pcb (KiCad board)
At the start: 2 copper layers, 144 x 160.4 mm, 81 parts, among them Q1 CRYSTAL, SW1 SW_PUSH, X1 RS-232, X2 P8000, X3 SD-CON, X4 PATA, X5 4_Pin_Molex, X6 P8000-Compact, X7 AVR-ISP-6

Commit message: update 3D and footprints
Parts:
- 1R4, 2R4, 3R4, R3, R6: footprint R1 -> Discret:R1
