File: P8000_WDC_Emulator/Hardware/P8000_WDC_Emulator.kicad_pcb (KiCad board)
At the start: 2 copper layers, 144 x 160.4 mm, 213 parts, among them Q1 CRYSTAL, SW1 SW_PUSH, X1 RS-232, X2 P8000, X3 SD-CON, X4 PATA, X5 4_Pin_Molex, X6 P8000-Compact, X7 AVR-ISP-6

Commit message: version 2.10
Parts:
- added R5: 4k7, Discret:R1, F.Cu at (148.6, 58.2)
- 1R4, 2R4: value 220 -> 300
Routing:
- net //RST2: track 113.0 -> 134.1 mm
Other:
- board text added: "P8000 WDC Emulator v 2.1.1 (c) Oliver Lehmann 2012, 2013, 2015, 2016 lehmann@ans-netz.de"
- board text removed: "P8000 WDC Emulator v 2.1 (c) Oliver Lehmann 2012, 2013, 2015, 2016 lehmann@ans-netz.de"
Changed lines of the file:
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@@
 (kicad_pcb (version 4) (host pcbnew 4.0.1-stable)
   (general
-    (links 361)
+    (links 363)
     (no_connects 0)
-    (area 19.428459 21.160739 163.809681 181.940201)
+    (area 16.002 11.8073 167.875258 181.940201)
     (thickness 1.6002)
-    (drawings 31)
-    (tracks 1526)
+    (drawings 33)
+    (tracks 1530)
     (zones 0)
-    (modules 213)
+    (modules 214)
     (nets 117)
   )
@@
   (title_block
     (title "P8000 WDC Emulator")
-    (date 2016-04-24)
-    (rev 2.1)
+    (date 2016-06-22)
+    (rev 2.1.1)
   )
   (layers
@@
       (effects (font (size 1 1) (thickness 0.15)))
     )
-    (fp_text value 220 (at -1.143 2.54 180) (layer F.Fab) hide
+    (fp_text value 300 (at -1.143 2.54 180) (layer F.Fab) hide
       (effects (font (size 1 1) (thickness 0.15)))
     )
@@
       (effects (font (size 1 1) (thickness 0.15)))
     )
-    (fp_text value 220 (at -1.143 2.54 180) (layer F.Fab) hide
+    (fp_text value 300 (at -1.143 2.54 180) (layer F.Fab) hide
       (effects (font (size 1 1) (thickness 0.15)))
     )
@@
       (net 41 GND) (clearance 0.00254) (zone_connect 2))
   )
+  (module Discret:R1 (layer Front)
+    (at 148.58 58.18 180)
+    (descr "Resistance verticale")
+    (tags R)
+    (fp_text reference R5 (at -1.016 2.54 180) (layer F.SilkS)
+      (effects (font (size 1 1) (thickness 0.15)))
+    )
+    (fp_text value 4k7 (at 1.42 2.87 180) (layer F.Fab) hide
+      (effects (font (size 1 1) (thickness 0.15)))
+    )
+    (fp_line (start -1.27 0) (end 1.27 0) (layer F.SilkS) (width 0.15))
+    (fp_circle (center -1.27 0) (end -0.635 1.27) (layer F.SilkS) (width 0.15))
+    (pad 1 thru_hole circle (at -1.27 0 180) (size 1.397 1.397) (drill 0.8128) (layers *.Cu *.Mask F.SilkS)
+      (net 5 //RST2))
+    (pad 2 thru_hole circle (at 1.27 0 180) (size 1.397 1.397) (drill 0.8128) (layers *.Cu *.Mask F.SilkS)
+      (net 42 VCC))
+    (model Discret.3dshapes/R1.wrl
+      (at (xyz 0 0 0))
+      (scale (xyz 1 1 1))
+      (rotate (xyz 0 0 0))
+    )
+  )
+  (gr_text 1 (at 23.29 79.09) (layer F.SilkS)
+    (effects (font (size 1.50114 1.00076) (thickness 0.25146)))
+  )
+  (gr_text 1 (at 76.43 36.61) (layer F.SilkS)
+    (effects (font (size 2.032 1.524) (thickness 0.3048)))
+  )
+  (gr_text 1 (at 76.44 29.24) (layer F.SilkS)
+    (effects (font (size 2.032 1.524) (thickness 0.3048)))
+  )
   (gr_line (start 80.645 61.214) (end 80.645 71.374) (angle 90) (layer F.SilkS) (width 0.381))
   (gr_line (start 139.065 61.214) (end 80.645 61.214) (angle 90) (layer F.SilkS) (width 0.381))
@@
     (effects (font (size 2.032 1.524) (thickness 0.3048)))
   )
-  (gr_text "P8000 WDC Emulator v 2.1\n(c) Oliver Lehmann 2012, 2013, 2015, 2016\nlehmann@ans-netz.de" (at 69.27596 77.65034) (layer F.SilkS)
+  (gr_text "P8000 WDC Emulator v 2.1.1\n(c) Oliver Lehmann 2012, 2013, 2015, 2016\nlehmann@ans-netz.de" (at 69.27596 77.65034) (layer F.SilkS)
     (effects (font (size 2.032 1.524) (thickness 0.3048)))
   )
@@
     (effects (font (size 1.80086 1.39954) (thickness 0.3048)) (justify left))
   )
-  (gr_text 1 (at 23.70074 79.14894) (layer F.SilkS)
-    (effects (font (size 0.8001 0.8001) (thickness 0.0889)))
-  )
   (gr_text 1 (at 54.51562 12.50072) (layer F.SilkS)
     (effects (font (size 0.8001 0.8001) (thickness 0.0889)))
@@
     (effects (font (size 1.80086 1.39954) (thickness 0.3048)) (justify left))
   )
-  (gr_text 1 (at 22.86 161.29) (layer F.SilkS)
+  (gr_text 1 (at 23.36 161.52) (layer F.SilkS)
     (effects (font (size 1.50114 1.00076) (thickness 0.25146)))
   )
@@
   (segment (start 78.74 27.305) (end 78.74 29.93) (width 0.2032) (layer Back) (net 4))
   (segment (start 78.74 34.925) (end 78.362202 34.925) (width 0.2032) (layer Back) (net 4))
+  (segment (start 142.24 76.2) (end 147.97 70.47) (width 0.2032) (layer Front) (net 5))
+  (segment (start 149.85 63.01) (end 149.85 58.18) (width 0.2032) (layer Front) (net 5))
+  (segment (start 147.97 64.89) (end 149.85 63.01) (width 0.2032) (layer Front) (net 5))
+  (segment (start 147.97 70.47) (end 147.97 64.89) (width 0.2032) (layer Front) (net 5))
   (segment (start 117.39 41.27) (end 117.61 41.27) (width 0.2032) (layer Back) (net 5))
   (segment (start 119.66 35.57) (end 120.5 35.57) (width 0.2032) (layer Back) (net 5))
